File: Eagle_Project/RASP_GPIO_DAC_ADC_2.sch (EAGLE design)
At the start: 159 parts, among them U1 MCP23008-E/P, U2 MCP23008-E/P, U3 MCP4728-E/UN, U4 MCP23008-E/P, U5 MCP23008-E/P

Commit message: Insert DCDC in schematic and make a sheet for components
Parts:
- added C52, C53, C54: 1uF, capacitor-wima:C2,5-3
- added C_IN, C_IN1, C_OUT, C_OUT1: 680uF, rcl:CPOL-EU085CS-1AR
- added D53, D58: DIODE-ZENER5.6V, SparkFun-DiscreteSemi:DIODE-ZENER5.6V
- added D59, D62: 5.1V, SparkFun-DiscreteSemi:DIODE-ZENER5.6V
- added D60, D61: 2.2V, SparkFun-DiscreteSemi:DIODE-ZENER5.6V
- added IC1, IC2: LM2596S, national-semiconductor:LM2596S
- added L1, L2: (no value), rcl:L-US0204/5
- added R57, R60: 1K, resistor:R-EU_0204/2V
- added R58, R59: 100K, resistor:R-EU_0204/2V
- added R_PULLUP_SCL, R_PULLUP_SDA: 10K, resistor:R-EU_0204/2V
- added U$4: MCP3428-E/SL, Microchip_By_element14_Batch_1:MCP3428-E/SL
- added U8: MCP23008-E/P, Microchip_By_element14_Batch_1:MCP23008-E/P
- added U9: MCP4728-E/UN, Microchip_By_element14_Batch_1:MCP4728-E/UN
Connections:
- removed net N$1: U$1.SCL, U$3.SCL, U1.SCL, U2.SCL, U3.SCL, U4.SCL, U5.SCL
- new net N$122: D58.C, IC2.OUT, L2.1
- new net N$123: D59.C, R57.2
- new net N$124: R57.1
- new net N$125: C52.1, D60.C, R58.2
- new net N$126: R58.1
- new net N$127: C53.2, D61.C, R59.2
- new net N$128: R59.1
- new net N$129: C54.1, D62.C, R60.2
- new net N$130: R60.1
- new net N$96: D53.C, IC1.OUT, L1.1
- new net N$98: R_PULLUP_SCL.1, U$1.SCL, U$3.SCL, U1.SCL, U2.SCL, U3.SCL, U4.SCL, U5.SCL
- net GND: now also C52.2, C53.1, C54.2, C_IN.-, C_IN1.-, C_OUT.-, C_OUT1.-, D53.A, D58.A, D59.A, D60.A, D61.A, D62.A, IC1.!ON!/OFF, IC1.GND, IC2.!ON!/OFF, IC2.GND
- net N$3: now also R_PULLUP_SDA.1
- net VDD: now also C_IN.+, C_IN1.+, C_OUT.+, C_OUT1.+, IC1.FB, IC1.VIN, IC2.FB, IC2.VIN, L1.2, L2.2, R_PULLUP_SCL.2, R_PULLUP_SDA.2
Other:
- note added: "DCDC Power supply"

Commit message: Update schematics
Parts:
- C_OUT, C_OUT1: value 680uF -> 220uF
- D53, D58: value DIODE-ZENER5.6V -> 1N5824
- L1, L2: value (none) -> 33uH
Changed lines of the file:
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@@
 <part name="VDD1" library="supply1" deviceset="VDD" device="" value="VDD 12V"/>
 <part name="C_IN" library="rcl" deviceset="CPOL-EU" device="085CS-1AR" value="680uF"/>
-<part name="D53" library="SparkFun-DiscreteSemi" deviceset="DIODE-ZENER" device="5.6V" value=""/>
-<part name="L1" library="rcl" deviceset="L-US" device="0204/5"/>
-<part name="C_OUT" library="rcl" deviceset="CPOL-EU" device="085CS-1AR" value="680uF"/>
+<part name="D53" library="SparkFun-DiscreteSemi" deviceset="DIODE-ZENER" device="5.6V" value="1N5824"/>
+<part name="L1" library="rcl" deviceset="L-US" device="0204/5" value="33uH"/>
+<part name="C_OUT" library="rcl" deviceset="CPOL-EU" device="085CS-1AR" value="220uF"/>
 <part name="SUPPLY11" library="SparkFun-Aesthetics" deviceset="VDD" device=""/>
 <part name="SUPPLY12" library="SparkFun-Aesthetics" deviceset="VDD" device=""/>
@@
 <part name="VDD2" library="supply1" deviceset="VDD" device="" value="VDD 12V"/>
 <part name="C_IN1" library="rcl" deviceset="CPOL-EU" device="085CS-1AR" value="680uF"/>
-<part name="D58" library="SparkFun-DiscreteSemi" deviceset="DIODE-ZENER" device="5.6V" value=""/>
-<part name="L2" library="rcl" deviceset="L-US" device="0204/5"/>
-<part name="C_OUT1" library="rcl" deviceset="CPOL-EU" device="085CS-1AR" value="680uF"/>
+<part name="D58" library="SparkFun-DiscreteSemi" deviceset="DIODE-ZENER" device="5.6V" value="1N5824"/>
+<part name="L2" library="rcl" deviceset="L-US" device="0204/5" value="33uH"/>
+<part name="C_OUT1" library="rcl" deviceset="CPOL-EU" device="085CS-1AR" value="220uF"/>
 <part name="SUPPLY13" library="SparkFun-Aesthetics" deviceset="VDD" device=""/>
 <part name="R57" library="resistor" deviceset="R-EU_" device="0204/2V" value="1K"/>
